File: kicad/C64 RF Modulator Replacement.kicad_pcb (KiCad board)
At the start: 2 copper layers, 51.8 x 32.6 mm, 33 parts, among them J1 Conn_01x04_Male, J2 Conn_01x04_Male, Q1 BC547, Q2 BC547, U1 78L05

Commit message: Rev C
Parts:
- R4: value 33 -> 68
- RV1, RV2: footprint Potentiometer_THT:Potentiometer_Bourns_3296Y_Vertical -> Potentiometer_THT:Potentiometer_Bourns_3296W_Vertical
- moved JP6 3.62 mm to (182.4, 127.8)
- moved JP7 3.62 mm to (187.9, 127.8)
- moved R4 3.43 mm to (182.0, 115.3)
- moved R5 3.30 mm to (182.0, 111.9)
- moved RV1 1.27 mm to (184.7, 123.2)
- moved RV2 1.27 mm to (190.3, 123.2)
Routing:
- net ChromaOut: track 22.3 -> 28.7 mm
- net Net-(C6-Pad1): track 32.1 -> 29.5 mm
- net Net-(JP7-Pad1): track 16.1 -> 14.0 mm
- net Net-(JP6-Pad1): track 17.4 -> 15.6 mm

Commit message: Rev D
Parts:
- RV1, RV2: footprint Potentiometer_THT:Potentiometer_Bourns_3296W_Vertical -> C64 RF Modulator Replacement:Potentiometer_Bourns_3296W_Vertical
- moved D2 0.25 mm to (221.6, 129.2)
Routing:
- net GND: vias 2 -> 12
Other:
- net class Power: trace_width 0.5 -> 0.4
- board text added: "Rev D"
- board text removed: "Rev C"
