File: kicad/C64 RF Modulator Replacement.sch (KiCad schematic (older format))
At the start: 33 parts, among them J1 Conn_01x04_Male, J2 Conn_01x04_Male, Q1 BC547, Q2 BC547, U1 78L05

Commit message: Rev C
Parts:
- RV1: footprint Potentiometer_THT:Potentiometer_Bourns_3296Y_Vertical -> Potentiometer_THT:Potentiometer_Bourns_3296W_Vertical
- RV2: value 250 -> 220; footprint Potentiometer_THT:Potentiometer_Bourns_3296Y_Vertical -> Potentiometer_THT:Potentiometer_Bourns_3296W_Vertical
Other:
- note removed: "200Ω or 220Ω can be \nsubstituted for RV2 if neecesary"
- moved on the sheet: C1, C6, D2, JP6, JP7, L2, Q1, Q2, R1, R11, R12, R2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

Commit message: Rev D
Parts:
- RV1, RV2: footprint Potentiometer_THT:Potentiometer_Bourns_3296W_Vertical -> C64 RF Modulator Replacement:Potentiometer_Bourns_3296W_Vertical
Changed lines of the file:
@@
 Sheet 1 1
 Title "C64 RF Modulator Replacement"
-Date "2020-04-05"
+Date "2020-04-07"
 Rev "C"
 Comp "mbarszcz-pcb"
@@
 F 0 "RV1" V 8625 2525 50  0000 C CNN
 F 1 "1K" V 8725 2525 50  0000 C CNN
-F 2 "Potentiometer_THT:Potentiometer_Bourns_3296W_Vertical" H 8725 2525 50  0001 C CNN
+F 2 "C64 RF Modulator Replacement:Potentiometer_Bourns_3296W_Vertical" H 8725 2525 50  0001 C CNN
 F 3 "~" H 8725 2525 50  0001 C CNN
 	1    8725 2525
@@
 F 0 "RV2" V 8125 4000 50  0000 C CNN
 F 1 "220" V 8220 4000 50  0000 C CNN
-F 2 "Potentiometer_THT:Potentiometer_Bourns_3296W_Vertical" H 8225 4000 50  0001 C CNN
+F 2 "C64 RF Modulator Replacement:Potentiometer_Bourns_3296W_Vertical" H 8225 4000 50  0001 C CNN
 F 3 "~" H 8225 4000 50  0001 C CNN
 	1    8225 4000
